Commit message: added full urdf

File: urdf-assembly.urdf (robot description, URDF)
Before this commit: robot urdf-assembly, 3 links, 2 joints
Links:
- added link left_back_knee, mass 0.39133711147367384; collision mesh filename=meshes/left_back_knee.stl scale=0.001 0.001 0.001; visual mesh filename=meshes/left_back_knee.stl scale=0.001 0.001 0.001
- added link left_back_leg, mass 0.28781330300213154; collision mesh filename=meshes/left_back_leg.stl scale=0.001 0.001 0.001; visual mesh filename=meshes/left_back_leg.stl scale=0.001 0.001 0.001
- added link left_front_knee, mass 0.39133711147367384; collision mesh filename=meshes/left_front_knee.stl scale=0.001 0.001 0.001; visual mesh filename=meshes/left_front_knee.stl scale=0.001 0.001 0.001
- added link left_front_leg, mass 0.28781330300213154; collision mesh filename=meshes/left_front_leg.stl scale=0.001 0.001 0.001; visual mesh filename=meshes/left_front_leg.stl scale=0.001 0.001 0.001
- added link right_front_knee, mass 0.39133711148958433; collision mesh filename=meshes/right_front_knee.stl scale=0.001 0.001 0.001; visual mesh filename=meshes/right_front_knee.stl scale=0.001 0.001 0.001
- added link right_front_leg, mass 0.28781330300213154; collision mesh filename=meshes/right_front_leg.stl scale=0.001 0.001 0.001; visual mesh filename=meshes/right_front_leg.stl scale=0.001 0.001 0.001
Joints:
- added joint base-combined-v1_Revolute-11: type continuous, parent base-combined-v1, child left_back_leg, origin xyz=-0.12649499 0.04622836 -0.07920745 rpy=3.1415926535897922 -0.0 0.0, axis 0.0 -8.500145032286205e-16 1.0
- added joint base-combined-v1_Revolute-7: type continuous, parent base-combined-v1, child right_front_leg, origin xyz=0.10350501 0.04622836 0.07744255 rpy=-3.1415926535897927 -0.0 0.0, axis 0.0 7.598088824778261e-16 1.0
- added joint base-combined-v1_Revolute-9: type continuous, parent base-combined-v1, child left_front_leg, origin xyz=0.10350501 0.04622836 -0.07920745 rpy=3.1415926535897922 -0.0 0.0, axis 0.0 -8.500145032286205e-16 1.0
- added joint left_back_leg_Revolute-12: type continuous, parent left_back_leg, child left_back_knee, origin xyz=-0.09187012000000003 0.09218367000000001 0.010300000000000064 rpy=-3.1415926535897922 -3.900666110763166e-45 4.58894065447968e-30, axis 0.0 -0.0 -1.0000000000000002
- added joint left_front_leg_Revolute-10: type continuous, parent left_front_leg, child left_front_knee, origin xyz=-0.09187012000000003 0.09218367000000001 0.010300000000000064 rpy=-3.1415926535897922 1.9721522630524905e-31 4.588940654479647e-30, axis -1.9721522630525295e-31 -3.944304526105059e-31 -1.0
- added joint right_front_leg_Revolute-8: type continuous, parent right_front_leg, child right_front_knee, origin xyz=-0.09218367000000004 0.09187012 -0.010300000000000073 rpy=3.1415926535897927 3.944304526105023e-31 -4.7387042952618626e-30, axis 3.944304526105059e-31 3.944304526105059e-31 1.0
