Commit message: WIP: snapshot before laptop wipe
Co-Authored-By: Claude Sonnet 5.5 <noreply@anthropic.com>

File: urdf-assembly.urdf (robot description, URDF)
Before this commit: robot urdf-assembly, 9 links, 8 joints
Links:
- link base-combined-v1: mass 5.722096819893475 -> 1.5
- link left_back_knee: mass 0.39133711147367384 -> 0.1
- link left_back_leg: mass 0.28781330300213154 -> 0.1
- link left_front_knee: mass 0.39133711147367384 -> 0.1
- link left_front_leg: mass 0.28781330300213154 -> 0.1
- link right_back_knee: mass 0.39133711148958433 -> 0.1
- link right_back_leg: mass 0.28781330300213154 -> 0.1
- link right_front_knee: mass 0.39133711148958433 -> 0.1
- link right_front_leg: mass 0.28781330300213154 -> 0.1
